Commit message: different localizaiton configs added

File: src/ugv_sim/scout/scout_description/urdf/scout_v2.xacro (robot description, xacro)
@@ -31,5 +31,5 @@
   </joint>
   <joint name="camera_joint" type="fixed">
-    <origin xyz="0.5 0 0.1112" rpy="0 0 0"/>
+    <origin xyz="0 0 0.3" rpy="0 0.3 0"/>
     <parent link="base_link"/>
     <child link="camera_link"/>
